Commit message: feat(description): single complete URDF replacing system standard
The system turtlebot4_description publishes the standard turtlebot4 URDF
which puts rplidar at a fixed position relative to a 'shell_link' that
doesn't physically exist on our bare Create3. The two competing TF chains
(shell_link->rplidar_link from system, base_link->rplidar_link from us)
were resolving to the wrong position.

Solution: drop the dual-RSP approach. Our custom_tb4_description now
provides a SINGLE complete URDF that includes irobot_create_description's
create3.urdf.xacro and adds our sensors at correct physical positions.
The new install_description_override.sh patches the system standard.launch.py
to suppress its description include, leaving only ours active.

- urdf/custom_extras.urdf.xacro -> custom_robot.urdf.xacro (complete)
- description.launch.py: publishes /robot_description (canonical name)
                         + joint_state_publisher
- package.xml: depend on irobot_create_description, joint_state_publisher
- scripts/install_description_override.sh: patch /etc/ros/humble system file

File: src/custom_tb4_description/urdf/custom_robot.urdf.xacro (robot description, xacro)
@@ -1,15 +1,19 @@
 <?xml version="1.0"?>
 <!--
-  Custom extras URDF for our bare Create3 + RPLIDAR + USB camera setup.
-  This URDF is published by a SECOND robot_state_publisher (named custom_extras_rsp)
-  alongside the system's Create3 RSP. It only adds the sensor links, not Create3 base.
-  Mounting:
-    - RPLIDAR: 3cm behind dock-direction center, 12cm above base, yaw=-90deg
-              (triangle marker points to robot's left, scan direction = clockwise)
-    - Camera:  15cm behind center on aluminum pole, 42cm above base, facing forward
+  Complete URDF for our bare iRobot Create3 + custom-mounted RPLIDAR + USB camera.
+  This file is intended to REPLACE the system turtlebot4 robot_description
+  (which assumes the standard turtlebot4 shell + sensor mounts that we don't
+  have). It includes the official Create3 base model and adds our custom
+  sensor mounts at their actual physical positions.
+  Mounting (measured on the real robot):
+    - RPLIDAR A1: 3 cm behind dock-direction center, 12 cm above base,
+                  yaw = -pi/2 (triangle marker points to robot's left)
+    - USB camera: 15 cm behind center on aluminum pole, 42 cm above base,
+                  facing forward
+    - Aluminum pole: visual only, 1 cm radius, 42 cm long
 -->
-<robot xmlns:xacro="http://ros.org/wiki/xacro" name="custom_extras">
-  <!-- base_link is a placeholder; Create3's RSP also publishes it -->
-  <link name="base_link"/>
+<robot name="custom_tb4" xmlns:xacro="http://ros.org/wiki/xacro">
+  <!-- ===== Create3 base ===== -->
+  <xacro:include filename="$(find irobot_create_description)/urdf/create3.urdf.xacro" />
   <!-- ===== RPLIDAR ===== -->
   <joint name="rplidar_joint" type="fixed">
@@ -34,5 +38,5 @@
     </inertial>
   </link>
-  <!-- ===== Aluminum pole (visual only) ===== -->
+  <!-- ===== Aluminum pole (visual only, holds the camera) ===== -->
   <joint name="pole_joint" type="fixed">
     <parent link="base_link"/>
@@ -50,6 +54,10 @@
       </material>
     </visual>
+    <inertial>
+      <mass value="0.05"/>
+      <inertia ixx="0.0001" ixy="0" ixz="0" iyy="0.0001" iyz="0" izz="0.0001"/>
+    </inertial>
   </link>
-  <!-- ===== USB Camera ===== -->
+  <!-- ===== USB camera ===== -->
   <joint name="camera_joint" type="fixed">
     <parent link="base_link"/>
